File: 01 - TSTE 2025&2026/Old DAQ Refinement/Analog Input Rev B/KiCad PCB Files/AI_Board_Rev_B.kicad_pcb (KiCad board)
At the start: 2 copper layers, 130 x 165 mm, 54 parts, among them J1 DC37_Socket_MountingHoles, J10 AI4 M12, J11 AI4 XT30, J12 AI5 M12, J13 AI5 XT30, J14 AI6 M12, J15 AI6 XT30, J16 AI7 M12, J17 AI7 XT30, J18 AI8 M12, J19 AI8 XT30, J2 AI0 M12, J20 AI9 M12, J21 AI9 XT30, J22 AI10 M12, J23 AI10 XT30, J24 AI11 M12, J25 AI11 XT30, J26 AI12 M12, J27 AI12 XT30, J28 AI13 M12, J29 AI13 XT30, J3 AI0 XT30, J30 AI14 M12, J31 AI14 XT30, J32 AI15 M12, J33 AI15 XT30, J4 AI1 M12, J5 AI1 XT30, J6 AI2 M12, J7 AI2 XT30, J8 AI3 M12, J9 AI3 XT30, M3 MountingHole_3.2mm_M3

Commit message: Add files via upload
Connections:
- J1 pad 1: /NC -> GND
- J10 pad 4: Net-(J10-Pin_4) -> GND
- J11 pad 1: Net-(J10-Pin_4) -> GND
- J12 pad 4: Net-(J12-Pin_4) -> GND
- J13 pad 1: Net-(J12-Pin_4) -> GND
- J14 pad 4: Net-(J14-Pin_4) -> GND
- J15 pad 1: Net-(J14-Pin_4) -> GND
- J16 pad 4: Net-(J16-Pin_4) -> GND
- J17 pad 1: Net-(J16-Pin_4) -> GND
- J18 pad 4: Net-(J18-Pin_4) -> GND
- J19 pad 1: Net-(J18-Pin_4) -> GND
- J2 pad 4: Net-(J2-Pin_4) -> GND
- J20 pad 4: Net-(J20-Pin_4) -> GND
- J21 pad 1: Net-(J20-Pin_4) -> GND
- J22 pad 4: Net-(J22-Pin_4) -> GND
- J23 pad 1: Net-(J22-Pin_4) -> GND
- J24 pad 4: Net-(J24-Pin_4) -> GND
- J25 pad 1: Net-(J24-Pin_4) -> GND
- J26 pad 4: Net-(J26-Pin_4) -> GND
- J27 pad 1: Net-(J26-Pin_4) -> GND
- J28 pad 4: Net-(J28-Pin_4) -> GND
- J29 pad 1: Net-(J28-Pin_4) -> GND
- J3 pad 1: Net-(J2-Pin_4) -> GND
- J30 pad 4: Net-(J30-Pin_4) -> GND
- J31 pad 1: Net-(J30-Pin_4) -> GND
- J32 pad 4: Net-(J32-Pin_4) -> GND
- J33 pad 1: Net-(J32-Pin_4) -> GND
- J4 pad 4: Net-(J4-Pin_4) -> GND
- J5 pad 1: Net-(J4-Pin_4) -> GND
- J6 pad 4: Net-(J6-Pin_4) -> GND
- J7 pad 1: Net-(J6-Pin_4) -> GND
- J8 pad 4: Net-(J8-Pin_4) -> GND
- J9 pad 1: Net-(J8-Pin_4) -> GND
- R1 pad 2: Net-(J2-Pin_4) -> GND
- R10 pad 2: Net-(J20-Pin_4) -> GND
- R11 pad 2: Net-(J22-Pin_4) -> GND
- R12 pad 2: Net-(J24-Pin_4) -> GND
- R13 pad 2: Net-(J26-Pin_4) -> GND
- R14 pad 2: Net-(J28-Pin_4) -> GND
- R15 pad 2: Net-(J30-Pin_4) -> GND
- R16 pad 2: Net-(J32-Pin_4) -> GND
- R2 pad 2: Net-(J4-Pin_4) -> GND
- R3 pad 2: Net-(J6-Pin_4) -> GND
- R4 pad 2: Net-(J8-Pin_4) -> GND
- R5 pad 2: Net-(J10-Pin_4) -> GND
- R6 pad 2: Net-(J12-Pin_4) -> GND
- R7 pad 2: Net-(J14-Pin_4) -> GND
- R8 pad 2: Net-(J16-Pin_4) -> GND
- R9 pad 2: Net-(J18-Pin_4) -> GND
Routing:
- net GND: track 0.00 -> 600.9 mm
- net Net-(J8-Pin_4): track 38.4 -> 0.00 mm
- net Net-(J24-Pin_4): track 38.4 -> 0.00 mm
- net Net-(J16-Pin_4): track 38.4 -> 0.00 mm
- net Net-(J18-Pin_4): track 37.5 -> 0.00 mm
- net Net-(J6-Pin_4): track 37.4 -> 0.00 mm
- net Net-(J4-Pin_4): track 37.4 -> 0.00 mm
- net Net-(J30-Pin_4): track 37.4 -> 0.00 mm
- net Net-(J28-Pin_4): track 37.4 -> 0.00 mm
- net Net-(J26-Pin_4): track 37.4 -> 0.00 mm
- net Net-(J20-Pin_4): track 37.4 -> 0.00 mm
- net Net-(J22-Pin_4): track 37.4 -> 0.00 mm
- net Net-(J2-Pin_4): track 37.4 -> 0.00 mm
- net Net-(J14-Pin_4): track 37.4 -> 0.00 mm
- net Net-(J12-Pin_4): track 37.4 -> 0.00 mm
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- added copper zone on B.Cu, net GND
- added copper zone on F.Cu, net GND
Other:
- board text added: "AI Board"
- board text added: "Rev_B"
- board text removed: "Analog Input Board Rev. B Isaac Lough 10/6/25"
