File: 01 - TSTE 2025&2026/Old DAQ Refinement/Analog Input Rev B/KiCad PCB Files/AI_Board_Rev_B.kicad_sch (KiCad schematic)
At the start: 49 parts, among them J1 DC37_Socket_MountingHoles, J10 AI4 M12, J11 AI4 XT30, J12 AI5 M12, J13 AI5 XT30, J14 AI6 M12, J15 AI6 XT30, J16 AI7 M12, J17 AI7 XT30, J18 AI8 M12, J19 AI8 XT30, J2 AI0 M12, J20 AI9 M12, J21 AI9 XT30, J22 AI10 M12, J23 AI10 XT30, J24 AI11 M12, J25 AI11 XT30, J26 AI12 M12, J27 AI12 XT30, J28 AI13 M12, J29 AI13 XT30, J3 AI0 XT30, J30 AI14 M12, J31 AI14 XT30, J32 AI15 M12, J33 AI15 XT30, J4 AI1 M12, J5 AI1 XT30, J6 AI2 M12, J7 AI2 XT30, J8 AI3 M12, J9 AI3 XT30

Commit message: Add files via upload
Connections:
- net NC is gone; now on net GND: J1.1
- net GND: now reaches J18.4 (Pin_4), J19.1 (Pin_1), R9.2
- net GND: now also J10.4 (Pin_4), J11.1 (Pin_1), J12.4 (Pin_4), J13.1 (Pin_1), J14.4 (Pin_4), J15.1 (Pin_1), J16.4 (Pin_4), J17.1 (Pin_1), J2.4 (Pin_4), J20.4 (Pin_4), J21.1 (Pin_1), J22.4 (Pin_4), J23.1 (Pin_1), J24.4 (Pin_4), J25.1 (Pin_1), J26.4 (Pin_4), J27.1 (Pin_1), J28.4 (Pin_4), J29.1 (Pin_1), J3.1 (Pin_1), J30.4 (Pin_4), J31.1 (Pin_1), J32.4 (Pin_4), J33.1 (Pin_1), J4.4 (Pin_4), J5.1 (Pin_1), J6.4 (Pin_4), J7.1 (Pin_1), J8.4 (Pin_4), J9.1 (Pin_1), R1.2, R10.2, R11.2, R12.2, R13.2, R14.2, R15.2, R16.2, R2.2, R3.2, R4.2, R5.2, R6.2, R7.2, R8.2
