File: 01 - TSTE 2025&2026/Old DAQ Refinement/Digital IO Rev B/Digital IO Board Rev B.kicad_pcb (KiCad board)
At the start: 2 copper layers, 85.5 x 77 mm, 22 parts, among them J1 DIO0 JST-VH, J10 DIO8 JST-VH, J11 DIO9 JST-VH, J12 DIO10 JST-VH, J13 DIO11 JST-VH, J14 DIO12 JST-VH, J15 DIO13 JST-VH, J16 DIO14 JST-VH, J17 DIO15 JST-VH, J2 DIO1 JST-VH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

Commit message: Final Files
Other:
- board text added: "October 2025"
Changed lines of the file:
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@@
 	)
 	(gr_text "Gibson Curtis"
-		(at 96.5 88.5 90)
+		(at 96.5 98 90)
 		(layer "F.SilkS")
 		(effects
@@
 		)
 	)
+	(gr_text "October 2025"
+		(at 96.5 78.5 90)
+		(layer "F.SilkS")
+		(effects
+			(font
+				(size 1.5 1.5)
+				(thickness 0.375)
+				(bold yes)
+			)
+			(justify left bottom)
+		)
+	)
 	(segment
 		(start 105 65)
@@
 		(hatch edge 0.5)
 		(connect_pads
-			(clearance 0.5)
-		)
-		(min_thickness 0.25)
-		(filled_areas_thickness no)
-		(fill yes
-			(thermal_gap 0.5)
-			(thermal_bridge_width 0.5)
-		)
-		(polygon
-			(pts
-				(xy 89 34.5) (xy 174.5 34.5) (xy 174.5 111.5) (xy 89 111.5)
-			)
-		)
-	)
-	(zone
-		(net 0)
-		(net_name "")
-		(layer "Edge.Cuts")
-		(hatch edge 0.5)
-		(connect_pads

Commit message: Vias Change Upload
Routing:
- net GND: vias 0 -> 66
Other:
- board text added: "{ "ViaStitching": "0.2", "stitch_zone_0": { "HSpacing": "8", "VSpacing": "8", "HOffset": "0", "VOffset": "0", "Clearance": "0.2", "Randomize": false } }"
